Commit message: added caster wheel

File: urdf/robot.urdf (robot description, URDF)
Before this commit: robot robot, 3 links, 2 joints
Links:
- added link link_caster_wheel, mass 1; collision sphere radius=0.25; visual sphere radius=0.125
Joints:
- added joint joint_caster_wheel: type fixed, parent link_chassis, child link_caster_wheel, origin xyz=0.8 0 -0.2 rpy=0 0 0
