Commit message: Created a simulated world featuring online/offline models and an animated actor

File: urdf/robot.xacro (robot description, xacro)
@@ -1,79 +1,5 @@
 <?xml version="1.0"?>
-<robot name="robot">
-<!-- Materials -->
-<gazebo reference="link_chassis">
-    <visual>
-        <material> <!-- Blue -->
-            <ambient>0.192 0.231 1.0 1.0</ambient>
-            <diffuse>0.482 0.682 1 1.0</diffuse>
-            <specular>0.0 0.01 1.0</specular>
-            <emissive>0.196 0.05 1 1.0</emissive>
-        </material>
-    </visual>
-</gazebo>
-<gazebo reference="link_caster_wheel">
-    <visual>
-        <material> <!-- Gray -->
-            <ambient>0.25 0.25 0.25 1.0</ambient>
-            <diffuse>0.25 0.25 0.25 1.0</diffuse>
-            <specular>0.0 0.0 0.0 1.0</specular>
-            <emissive>0.0 0.0 0.0 1.0</emissive>
-        </material>
-    </visual>
-    <collision>
-            <surface>
-                <friction>
-                    <ode>
-                        <mu>0.1</mu>
-                        <mu2>0.1</mu2>
-                    </ode>
-                </friction>
-            </surface>
-        </collision>
-</gazebo>
-<gazebo reference="link_left_wheel">
-    <visual>
-        <material> <!-- Black -->
-            <ambient>0.1 0.1 0.1 1.0</ambient>
-            <diffuse>0.1 0.1 0.1 1.0</diffuse>
-            <specular>0.0 0.0 0.0 1.0</specular>
-            <emissive>0.0 0.0 0.0 1.0</emissive>
-        </material>
-    </visual>
-    <collision>
-        <surface>
-            <friction>
-                <ode>
-                    <mu>0.8</mu>
-                    <mu2>0.8</mu2>
-                </ode>
-            </friction>
-        </surface>
-    </collision>
-</gazebo>
-<gazebo reference="link_right_wheel">
-    <visual>
-        <material> <!-- Black -->
-            <ambient>0.1 0.1 0.1 1.0</ambient>
-            <diffuse>0.1 0.1 0.1 1.0</diffuse>
-            <specular>0.0 0.0 0.0 1.0</specular>
-            <emissive>0.0 0.0 0.0 1.0</emissive>
-        </material>
-    </visual>
-    <collision>
-        <surface>
-            <friction>
-                <ode>
-                    <mu>0.8</mu>
-                    <mu2>0.8</mu2>
-                </ode>
-            </friction>
-        </surface>
-    </collision>
-</gazebo>
-<!-- keep fixed joint links seperate-->
-<gazebo reference="joint_chassis_caster_wheel">
-        <preserveFixedJoint>true</preserveFixedJoint>
-</gazebo>
+<robot name="robot" xmlns:xacro="http://www.ros.org/wiki/xacro">
+    <xacro:include filename="$(find robot_description)/urdf/robot.gazebo" />
     <!-- Link - chassis -->
     <link name="link_chassis">
@@ -114,5 +40,5 @@
     </inertial>
     <collision>
-        <origin rpy="1.5707 0 0" xyz="0 0.18 0" />
+        <origin rpy="${pi/2} 0 0" xyz="0 0.18 0" />
         <geometry>
             <cylinder length="0.12" radius="0.4"/>
@@ -120,5 +46,5 @@
     </collision>
     <visual>
-        <origin rpy="1.5707 0 0" xyz="0 0.18 0" />
+        <origin rpy="${pi/2} 0 0" xyz="0 0.18 0" />
         <geometry>
             <mesh filename="package://robot_description/meshes/wheel.stl" />
@@ -133,5 +59,5 @@
     </visual>
     <collision>
-        <origin rpy="1.5707 0 0" xyz="0 0.06 0" />
+        <origin rpy="${pi/2} 0 0" xyz="0 0.06 0" />
         <geometry>
             <cylinder length="0.12" radius="0.08"/>
@@ -139,5 +65,5 @@
     </collision>
     <visual>
-        <origin rpy="1.5707 0 0" xyz="0 0.06 0" />
+        <origin rpy="${pi/2} 0 0" xyz="0 0.06 0" />
         <geometry>
             <cylinder length="0.12" radius="0.08"/>
@@ -162,5 +88,5 @@
     </inertial>
     <collision>
-        <origin rpy="-1.5707 0 0" xyz="0 -0.18 0" />
+        <origin rpy="${-pi/2} 0 0" xyz="0 -0.18 0" />
         <geometry>
             <cylinder length="0.12" radius="0.4"/>
@@ -168,5 +94,5 @@
     </collision>
     <visual>
-        <origin rpy="-1.5707 0 0" xyz="0 -0.18 0" />
+        <origin rpy="${-pi/2} 0 0" xyz="0 -0.18 0" />
         <geometry>
             <mesh filename="package://robot_description/meshes/wheel.stl" />
@@ -174,5 +100,5 @@
     </visual>
     <collision>
-        <origin rpy="-1.5707 0 0" xyz="0 -0.06 0" />
+        <origin rpy="${-pi/2} 0 0" xyz="0 -0.06 0" />
         <geometry>
             <cylinder length="0.12" radius="0.08"/>
@@ -180,5 +106,5 @@
     </collision>
     <visual>
-        <origin rpy="-1.5707 0 0" xyz="0 -0.06 0" />
+        <origin rpy="${-pi/2} 0 0" xyz="0 -0.06 0" />
         <geometry>
             <cylinder length="0.12" radius="0.08"/>
@@ -227,28 +153,4 @@
     </visual>
 </link>
-<!-- Differential Drive Plugin -->
-<gazebo>
-    <plugin
-        filename="libignition-gazebo-diff-drive-system.so"
-        name="ignition::gazebo::systems::DiffDrive">
-        <left_joint>joint_chassis_left_wheel</left_joint>
-        <right_joint>joint_chassis_right_wheel</right_joint>
-        <wheel_separation>1.66</wheel_separation>
-        <wheel_radius>0.4</wheel_radius>
-        <odom_publish_frequency>20</odom_publish_frequency>
-        <topic>cmd_vel</topic>
-        <odom_topic>odom</odom_topic>
-        <tf_topic>tf</tf_topic>
-        <frame_id>odom</frame_id>
-        <child_frame_id>link_chassis</child_frame_id>
-    </plugin>
-</gazebo>
-<!-- Gazebo tags - Laser scan -->
-<gazebo reference="joint_laser_scan_chassis">
-    <preserveFixedJoint>true</preserveFixedJoint>
-</gazebo>
-<gazebo reference="link_laser_scan">
-    <material>Gazebo/DarkGrey</material>
-</gazebo>
 <!-- Laser scan -->
 <joint name="joint_laser_scan_chassis" type="fixed">
@@ -280,55 +182,3 @@
     </collision>
 </link>
-<!-- Laser Scanner Plugin -->
-<gazebo>
-    <plugin
-      filename="libignition-gazebo-sensors-system"
-      name="ignition::gazebo::systems::Sensors">
-      <!-- use ogre2 if ogre v2.x is installed, otherwise use ogre -->
-      <render_engine>ogre2</render_engine>
-    </plugin>
-</gazebo>
-<gazebo reference="link_laser_scan">
-    <sensor type="gpu_lidar" name="head_hokuyo_sensor">
-        <pose relative_to='lidar_frame'>0 0 0 0 0 0</pose>
-        <always_on>1</always_on>
-        <visualize>true</visualize>
-        <update_rate>20</update_rate>
-        <topic>/laser/scan</topic>
-        <ray>
-            <scan>
-                <horizontal>
-                    <samples>720</samples>
-                    <resolution>1</resolution>
-                    <min_angle>-1.570796</min_angle>
-                    <max_angle>1.570796</max_angle>
-                </horizontal>
-            </scan>
-            <range>
-                <min>0.20</min>
-                <max>10.0</max>
-                <resolution>0.01</resolution>
-            </range>
-            <noise>
-                <type>gaussian</type>
-                <mean>0.0</mean>
-                <stddev>0.01</stddev>
-            </noise>
-        </ray>
-    </sensor>
-</gazebo>
-<!-- IMU Plugin -->
-<gazebo>
-    <plugin filename="libignition-gazebo-imu-system"
-        name="ignition::gazebo::systems::Imu">
-    </plugin>
-</gazebo>
-<gazebo reference="link_chassis">
-    <sensor name="imu_sensor" type="imu">
-        <always_on>1</always_on>
-        <update_rate>20</update_rate>
-        <visualize>true</visualize>
-        <topic>imu</topic>
-    </sensor>
-</gazebo>
 </robot>

Commit message: complete simulation featuring launch with .xacro robot model

File: urdf/robot.xacro (robot description, xacro)
@@ -2,12 +2,19 @@
 <robot name="robot" xmlns:xacro="http://www.ros.org/wiki/xacro">
     <xacro:include filename="$(find robot_description)/urdf/robot.gazebo" />
+    <!-- Parameters -->
+    <xacro:property name="chassis_mass" value="10" />
+    <!-- pi is already defined as a global varibale -->
+    <!-- <xacro:property name="pi" value="3.141592654" /> -->
     <!-- Link - chassis -->
     <link name="link_chassis">
         <inertial>
-            <mass value="10" />
+            <mass value="${chassis_mass}" />
             <origin xyz="0 0 0.3" rpy="0 0 0" />
             <inertia ixx="1.5417" ixy="0" ixz="0" iyy="3.467" iyz="0" izz="4.742" />
         </inertial>
         <collision>
+            <!-- <geometry>
+                <box size="2 1.3 0.4" />
+            </geometry> -->
             <geometry>
                 <mesh filename="package://robot_description/meshes/chassis.stl" />
@@ -18,167 +25,205 @@
                 <mesh filename="package://robot_description/meshes/chassis.stl" />
             </geometry>
+            <!-- <geometry>
+                <box size="2 1.3 0.4" />
+            </geometry> -->
+            <material name="DarkBlue">
+                <color rgba="0.2 0.2 0.4 1" />
+            </material>
+        </visual>
+    </link>
+    <!-- Joint - caster wheel -->
+    <joint name="joint_chassis_caster_wheel" type="fixed">
+        <origin rpy="0 0 0" xyz="0.8 0 -0.15" />
+        <child link="link_caster_wheel" />
+        <parent link="link_chassis" />
+        <joint_properties damping="1.0" friction="1.0" />
+    </joint>
+    <!-- Link - caster wheel -->
+    <link name="link_caster_wheel">
+        <inertial>
+            <mass value="1" />
+            <origin xyz="0 0 0" rpy="0 0 0" />
+            <inertia ixx="0.002526666666667" ixy="0" ixz="0" iyy="0.002526666666667" iyz="0" izz="0.005"/>
+        </inertial>
+        <!-- Caster wheel support -->
+        <collision>
+            <origin rpy="0 0 0" xyz="0 0 -0.03" />
+            <geometry>
+                <sphere radius="0.2" />
+            </geometry>
+        </collision>
+        <visual>
+            <origin rpy="0 0 0" xyz="0 0 -0.03" />
+            <geometry>
+                <sphere radius="0.2" />
+            </geometry>
+            <material name="DarkBlue">
+                <color rgba="0.2 0.2 0.4 1" />
+            </material>
+        </visual>
+        <!-- Caster wheel -->
+        <collision>
+            <origin rpy="0 0 0" xyz="0 0 -0.15" />
+            <geometry>
+                <sphere radius="0.10" />
+            </geometry>
+        </collision>
+        <visual>
+            <origin rpy="0 0 0" xyz="0 0 -0.15" />
+            <geometry>
+                <sphere radius="0.10" />
+            </geometry>
+            <material name="Grey">
+                <color rgba="0.6 0.6 0.6 1" />
+            </material>
+        </visual>
+    </link>
+    <!-- Joint - chassis / left wheel -->
+    <joint name="joint_chassis_left_wheel" type="continuous">
+        <origin rpy="0 0 0" xyz="-0.5 0.65 0" />
+        <child link="link_left_wheel" />
+        <parent link="link_chassis" />
+        <axis rpy="0 0 0" xyz="0 1 0" />
+        <limit effort="10000" velocity="1000" />
+        <joint_properties damping="1.0" friction="1.0" />
+    </joint>
+    <!-- Link - left wheel -->
+    <link name="link_left_wheel">
+        <inertial>
+            <mass value="1" />
+            <origin xyz="0 0 0" rpy="0 0 0" />
+            <inertia ixx="0.002526666666667" ixy="0" ixz="0" iyy="0.002526666666667" iyz="0" izz="0.005"/>
+        </inertial>
+        <!-- Tires -->
+        <collision>
+            <origin rpy="${pi/2} 0 0" xyz="0 0.18 0" />
+            <geometry>
+                <cylinder length="0.12" radius="0.4"/>
+            </geometry>
+        </collision>
+        <visual>
+            <origin rpy="${pi/2} 0 0" xyz="0 0.18 0" />
+            <geometry>
+                <mesh filename="package://robot_description/meshes/wheel.stl" />
+            </geometry>
+            <material name="Black">
+                <color rgba="0.1 0.1 0.1 1" />
+            </material>
+        </visual>
+        <!-- Axle -->
+        <collision>
+            <origin rpy="${pi/2} 0 0" xyz="0 0.06 0" />
+            <geometry>
+                <cylinder length="0.12" radius="0.08"/>
+            </geometry>
+        </collision>
+        <visual>
+            <origin rpy="${pi/2} 0 0" xyz="0 0.06 0" />
+            <geometry>
+                <cylinder length="0.12" radius="0.08"/>
+            </geometry>
+            <material name="Grey">
+                <color rgba="0.6 0.6 0.6 1" />
+            </material>
+        </visual>
+        <!-- Hubcap -->
+        <visual>
+            <origin rpy="${pi/2} 0 0" xyz="0 0.18 0" />
+            <geometry>
+                <box size="0.02 0.5 0.02" />
+            </geometry>
+            <material name="Grey">
+                <color rgba="0.6 0.6 0.6 1" />
+            </material>
+        </visual>
+    </link>
+    <!-- Joint - chassis / right wheel -->
+    <joint name="joint_chassis_right_wheel" type="continuous">
+        <origin rpy="0 0 0" xyz="-0.5 -0.65 0" />
+        <child link="link_right_wheel" />
+        <parent link="link_chassis" />
+        <axis rpy="0 0 0" xyz="0 1 0" />
+        <limit effort="10000" velocity="1000" />
+        <joint_properties damping="1.0" friction="1.0" />
+    </joint>
+    <!-- Link - right wheel -->
+    <link name="link_right_wheel">
+        <inertial>
+            <mass value="1" />
+            <origin xyz="0 0 0" rpy="0 0 0" />
+            <inertia ixx="0.002526666666667" ixy="0" ixz="0" iyy="0.002526666666667" iyz="0" izz="0.005"/>
+        </inertial>
+        <!-- Tires -->
+        <collision>
+            <origin rpy="${pi/2} 0 0" xyz="0 -0.18 0" />
+            <geometry>
+                <cylinder length="0.12" radius="0.4"/>
+            </geometry>
+        </collision>
+        <visual>
+            <origin rpy="${pi/2} 0 0" xyz="0 -0.18 0" />
+            <geometry>
+                <mesh filename="package://robot_description/meshes/wheel.stl" />
+            </geometry>
+            <material name="Black">
+                <color rgba="0.1 0.1 0.1 1" />
+            </material>
+        </visual>
+        <!-- Axle -->
+        <collision>
+            <origin rpy="${pi/2} 0 0" xyz="0 -0.06 0" />
+            <geometry>
+                <cylinder length="0.12" radius="0.08"/>
+            </geometry>
+        </collision>
+        <visual>
+            <origin rpy="${pi/2} 0 0" xyz="0 -0.06 0" />
+            <geometry>
+                <cylinder length="0.12" radius="0.08"/>
+            </geometry>
+            <material name="Grey">
+                <color rgba="0.6 0.6 0.6 1" />
+            </material>
+        </visual>
+        <!-- Hubcap -->
+        <visual>
+            <origin rpy="${pi/2} 0 0" xyz="0 -0.18 0" />
+            <geometry>
+                <box size="0.02 0.5 0.02" />
+            </geometry>
+            <material name="Grey">
+                <color rgba="0.6 0.6 0.6 1" />
+            </material>
+        </visual>
+    </link>
+    <!-- Laser scan -->
+    <joint name="joint_laser_scan_chassis" type="fixed">
+        <origin rpy="0 0 0" xyz="0.8 0 0.3" />
+        <child link="link_laser_scan" />
+        <parent link="link_chassis" />
+        <joint_properties damping="1.0" friction="1.0" />
+    </joint>
+    <link name="link_laser_scan">
+        <inertial>
+            <origin xyz="0 0 0" rpy="0 0 0" />
+            <mass value="0.5" />
+            <inertia ixx="0.000252666666667" ixy="0" ixz="0" iyy="0.000252666666667" iyz="0" izz="0.0005"/>
+        </inertial>
+        <visual>
+            <origin xyz="0 0 0" rpy="0 0 0" />
+            <geometry>
+                <cylinder radius="0.15" length="0.20"/>
+            </geometry>
             <material name="Red">
-                <color rgba="1 0 0 1" />
-            </material>
-        </visual>
-    </link>
-    <!-- Joint - chassis / left wheel -->
-<joint name="joint_chassis_left_wheel" type="continuous">
-    <origin rpy="0 0 0" xyz="-0.5 0.65 0" />
-    <child link="link_left_wheel" />
-    <parent link="link_chassis" />
-    <axis rpy="0 0 0" xyz="0 1 0" />
-    <limit effort="10000" velocity="1000" />
-    <joint_properties damping="1.0" friction="1.0" />
-</joint>
-<!-- Link - left wheel -->
-<link name="link_left_wheel">
-    <inertial>
-        <mass value="1" />
-        <origin xyz="0 0 0" rpy="0 0 0" />
-        <inertia ixx="0.002526666666667" ixy="0" ixz="0" iyy="0.002526666666667" iyz="0" izz="0.005"/>
-    </inertial>
-    <collision>
-        <origin rpy="${pi/2} 0 0" xyz="0 0.18 0" />
-        <geometry>
-            <cylinder length="0.12" radius="0.4"/>
-        </geometry>
-    </collision>
-    <visual>
-        <origin rpy="${pi/2} 0 0" xyz="0 0.18 0" />
-        <geometry>
-            <mesh filename="package://robot_description/meshes/wheel.stl" />
-        </geometry>
-    </visual>
-    <!--Hubcap-->
-    <visual>
-        <origin rpy="0 0 0" xyz="0 0.18 0" />
-        <geometry>
-            <box size="0.05 0.05 0.5" />
-        </geometry>
-    </visual>
-    <collision>
-        <origin rpy="${pi/2} 0 0" xyz="0 0.06 0" />
-        <geometry>
-            <cylinder length="0.12" radius="0.08"/>
-        </geometry>
-    </collision>
-    <visual>
-        <origin rpy="${pi/2} 0 0" xyz="0 0.06 0" />
-        <geometry>
-            <cylinder length="0.12" radius="0.08"/>
-        </geometry>
-    </visual>
-</link>
-    <!-- Joint - chassis / Right wheel -->
-<joint name="joint_chassis_right_wheel" type="continuous">
-    <origin rpy="0 0 0" xyz="-0.5 -0.65 0" />
-    <child link="link_right_wheel" />
-    <parent link="link_chassis" />
-    <axis rpy="0 0 0" xyz="0 1 0" />
-    <limit effort="10000" velocity="1000" />
-    <joint_properties damping="1.0" friction="1.0" />
-</joint>
-<!-- Link - Right wheel -->
-<link name="link_right_wheel">
-    <inertial>
-        <mass value="1" />
-        <origin xyz="0 0 0" rpy="0 0 0" />
-        <inertia ixx="0.002526666666667" ixy="0" ixz="0" iyy="0.002526666666667" iyz="0" izz="0.005"/>
-    </inertial>
-    <collision>
-        <origin rpy="${-pi/2} 0 0" xyz="0 -0.18 0" />
-        <geometry>
-            <cylinder length="0.12" radius="0.4"/>
-        </geometry>
-    </collision>
-    <visual>
-        <origin rpy="${-pi/2} 0 0" xyz="0 -0.18 0" />
-        <geometry>
-            <mesh filename="package://robot_description/meshes/wheel.stl" />
-        </geometry>
-    </visual>
-    <collision>
-        <origin rpy="${-pi/2} 0 0" xyz="0 -0.06 0" />
-        <geometry>
-            <cylinder length="0.12" radius="0.08"/>
-        </geometry>
-    </collision>
-    <visual>
-        <origin rpy="${-pi/2} 0 0" xyz="0 -0.06 0" />
-        <geometry>
-            <cylinder length="0.12" radius="0.08"/>
-        </geometry>
-    </visual>
-        <!--Hubcap-->
-    <visual>
-        <origin rpy="0 0 0" xyz="0 -0.18 0" />
-        <geometry>
-            <box size="0.05 0.05 0.5" />
-        </geometry>
-    </visual>
-</link>
-<!-- Joint - chassis / castor wheel -->
-<joint name="joint_caster_wheel" type="fixed">
-    <origin rpy="0 0 0" xyz="0.8 0 -0.2"/>
-    <child link="link_caster_wheel"/>
-    <parent link="link_chassis"/>
-</joint>
-<!-- Link - caster wheel -->
-<link name = "link_caster_wheel">
-    <inertial>
-        <mass value = "1"/>
-        <origin
-            xyz = "0 0 0"
-            rpy = "0 0 0" />
-        <inertia
-            ixx="1" ixy="0" ixz="0"
-            iyy="1" iyz="0" izz="1"/>
-    </inertial>
-    <collision>
-        <origin
-            xyz="0 0 0"
-            rpy="0 0 0" />
-        <geometry>
-            <sphere radius="0.25"/>
-        </geometry>
-    </collision>
-    <visual>
-        <origin
-            xyz="0 0 0"
-            rpy="0 0 0" />
-        <geometry>
-            <sphere radius="0.125"/>
-        </geometry>
-    </visual>
-</link>
-<!-- Laser scan -->
-<joint name="joint_laser_scan_chassis" type="fixed">
-    <origin rpy="0 0 0" xyz="0.8 0 0.3" />
-    <child link="link_laser_scan" />
-    <parent link="link_chassis" />
-    <joint_properties damping="1.0" friction="1.0" />
-</joint>
-<link name="link_laser_scan">
-    <inertial>
-        <origin xyz="0 0 0" rpy="0 0 0" />
-        <mass value="0.5" />
-        <inertia ixx="0.000252666666667" ixy="0" ixz="0" iyy="0.000252666666667" iyz="0" izz="0.0005"/>
-    </inertial>
-    <visual>
-        <origin xyz="0 0 0" rpy="0 0 0" />
-        <geometry>
-            <cylinder radius="0.15" length="0.20"/>
-        </geometry>
-        <material name="Red">
-            <color rgba="0.7 0.1 0.1 1" />
-        </material>
-    </visual>
-    <collision>
-        <origin xyz="0 0 0" rpy="0 0 0"/>
-        <geometry>
-            <cylinder radius="0.15" length="0.20"/>
-        </geometry>
-    </collision>
-</link>
+                <color rgba="0.7 0.1 0.1 1" />
+            </material>
+        </visual>
+        <collision>
+            <origin xyz="0 0 0" rpy="0 0 0"/>
+            <geometry>
+                <cylinder radius="0.15" length="0.20"/>
+            </geometry>
+        </collision>
+    </link>
 </robot>
