Commit message: Alternative robot build using meshes

File: install/robot_description/share/robot_description/urdf/robot.urdf (robot description, URDF)
Before this commit: robot robot, 4 links, 3 joints
Links:
- link link_left_wheel: geometry collision cylinder length=0.12 radius=0.08; collision cylinder length=0.12 radius=0.4
- link link_right_wheel: geometry collision cylinder length=0.12 radius=0.08; collision cylinder length=0.12 radius=0.4
